File: Seminar.kicad_sch (KiCad schematic)
At the start: 13 parts, among them SW1 SW_Push, SW2 SW_Push, U1 NUCLEO64-F446RE, U2 PCF8574AP

Commit message: A
Connections:
- net GND: now also U1.70 (AGND)
- no-connect marks 53 -> 52
Changed lines of the file:
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@@
+	)
+	(junction
+		(at 177.8 127)
+		(diameter 0)
+		(color 0 0 0 0)
 	)
 	(junction
@@
 	)
 	(junction
+		(at 88.9 127)
+		(diameter 0)
+		(color 0 0 0 0)
+	)
+	(junction
 		(at 147.32 162.56)
 		(diameter 0)
@@
 	)
 	(no_connect
-		(at 243.84 139.7)
-	)
-	(no_connect
 		(at 203.2 124.46)
 	)
@@
 		)
 	)
+	(bus
+		(pts
+			(xy 177.8 12.7) (xy 177.8 127)
+		)
+		(stroke
+			(width 0)
+			(type dash_dot)
+		)
+	)
 	(wire
 		(pts
@@
 		)
 	)
+	(bus
+		(pts
+			(xy 12.7 127) (xy 88.9 127)
+		)
+		(stroke
+			(width 0)
+			(type dash_dot)
+		)
+	)
 	(wire
 		(pts
@@
 		)
 	)
+	(bus
+		(pts
+			(xy 177.8 127) (xy 177.8 166.37)
+		)
+		(stroke
+			(width 0)
+			(type dash_dot)
+		)
+	)
 	(wire
 		(pts
@@
 		)
 	)
+	(bus
+		(pts
+			(xy 88.9 127) (xy 177.8 127)
+		)
+		(stroke
+			(width 0)
+			(type dash_dot)
+		)
+	)
 	(wire
 		(pts
@@
 			(width 0)
 			(type default)
+		)
+	)
+	(bus
+		(pts
+			(xy 88.9 127) (xy 88.9 198.12)
+		)
+		(stroke
+			(width 0)
+			(type dash_dot)
 		)
 	)
@@
 					(unit 1)
 				)
+			)
+		)
+	)
+	(symbol
+		(lib_id "power:GND")
+		(at 243.84 139.7 0)
+		(unit 1)
+		(exclude_from_sim no)
+		(in_bom yes)
+		(on_board yes)
+		(dnp no)
+		(fields_autoplaced yes)
+		(property "Reference" "#PWR04"
+			(at 243.84 146.05 0)
+			(effects
+				(font
+					(size 1.27 1.27)
+				)
+				(hide yes)
+			)
+		)
+		(property "Value" "GND"
+			(at 243.84 144.78 0)
+			(effects
+				(font
+					(size 1.27 1.27)
+				)
+			)
+		)
+		(property "Footprint" ""
+			(at 243.84 139.7 0)
+			(effects
+				(font
+					(size 1.27 1.27)
+				)
+				(hide yes)
+			)
+		)
+		(property "Datasheet" ""
+			(at 243.84 139.7 0)
+			(effects
+				(font
+					(size 1.27 1.27)
+				)
+				(hide yes)
+			)
+		)
+		(property "Description" "Power symbol creates a global label with name \"GND\" , ground"
+			(at 243.84 139.7 0)
+			(effects
+				(font
+					(size 1.27 1.27)
+				)
+				(hide yes)
+			)
+		)
+		(pin "1"
+		)
+		(instances
+			(project "Seminar"
+				(path "/d4435fee-4739-44d4-a9c2-48a7a11be2d1"
+					(reference "#PWR04")
+					(unit 1)
+				)

Commit message: PCB update
Parts:
- added H1, H2, H3, H4: MountingHole, MountingHole:MountingHole_5.5mm, symbol Mechanical:MountingHole
- D1, D2: footprint (none) -> LED_THT:LED_D5.0mm
- R1, R2, R3, R4, R5: footprint (none) -> Resistor_SMD:R_1206_3216Metric_Pad1.30x1.75mm_HandSolder; Manufacturer (none) -> ROYALOHM; Manufacturer part number (none) -> 1206S4F2001T5E
- RV1: footprint (none) -> Potentiometer_SMD:Potentiometer_ACP_CA6-VSMD_Vertical; Manufacturer (none) -> Bourns Inc.; Manufacturer part number (none) -> PDB181-GTR03-504A2
- SW1, SW2: footprint (none) -> Button_Switch_THT:SW_PUSH_6mm_H4.3mm; Manufacturer (none) -> microswitch TACT; Manufacturer part number (none) -> TACT-64N-F
Connections:
- no-connect marks 52 -> 60
Other:
- moved on the sheet: DS1, R1, RV1, U2

Commit message: Update Seminar 7.12.
Parts:
- added C1: 22u, Capacitor_THT:CP_Radial_D5.0mm_P2.00mm, symbol Device:C_Polarized
- added C2: 220u, Capacitor_THT:CP_Radial_D5.0mm_P2.00mm, symbol Device:C_Polarized
- added D3: 11DQ06TA, Diode_THT:D_DO-41_SOD81_P12.70mm_Horizontal, symbol Device:D_Schottky_Filled
- added J1: Screw_Terminal_01x02, TerminalBlock_MetzConnect:TerminalBlock_MetzConnect_Type011_RT05502HBLC_1x02_P5.00mm_Horizontal, symbol Connector:Screw_Terminal_01x02
- added L1: 330u, Inductor_THT:L_Radial_D7.2mm_P3.00mm_Murata_1700, symbol Device:L
- added U3: LM2574N-5, Package_DIP:DIP-8_W7.62mm, symbol Regulator_Switching:LM2574N-5
- DS1: Manufacturer (none) -> Wandisplay; Manufacturer part number (none) -> WC1602B0SGW6B-A1
- U1: Manufacturer (none) -> STMicroelectronics; Manufacturer part number (none) -> STM32F446RET6
- U2: Manufacturer (none) -> NXP; Manufacturer part number (none) -> PCF8574AP,112
Connections:
- net +5V: now also C2.1, L1.2, U3.1 (FB)
- net GND: now also C1.2, C2.2, D3.2 (A), J1.1 (Pin_1), U3.2 (SGND), U3.3 (~{ON}/OFF), U3.4 (PGND)
- new net: D3.1 (K), L1.1, U3.7 (OUT)
- new net VD: C1.1, J1.2 (Pin_2), U3.5 (VIN)
Other:
- moved on the sheet: DS1, R1, RV1, U2

Commit message: Update Seminar 7.12. dva
Parts:
- RV1: footprint Potentiometer_SMD:Potentiometer_ACP_CA6-VSMD_Vertical -> Potentiometer_THT:Potentiometer_Bourns_3299Y_Vertical
Changed lines of the file:
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@@
 			)
 		)
-		(property "Footprint" "Potentiometer_SMD:Potentiometer_ACP_CA6-VSMD_Vertical"
+		(property "Footprint" "Potentiometer_THT:Potentiometer_Bourns_3299Y_Vertical"
 			(at 99.06 78.74 0)
 			(effects

Commit message: Baterija i Step up
Parts:
- removed C1: 22u, Capacitor_THT:CP_Radial_D5.0mm_P2.00mm, symbol Device:C_Polarized
- removed C2: 220u, Capacitor_THT:CP_Radial_D5.0mm_P2.00mm, symbol Device:C_Polarized
- removed D3: 11DQ06TA, Diode_THT:D_DO-41_SOD81_P12.70mm_Horizontal, symbol Device:D_Schottky_Filled
- removed J1: Screw_Terminal_01x02, TerminalBlock_MetzConnect:TerminalBlock_MetzConnect_Type011_RT05502HBLC_1x02_P5.00mm_Horizontal, symbol Connector:Screw_Terminal_01x02
- removed L1: 330u, Inductor_THT:L_Radial_D7.2mm_P3.00mm_Murata_1700, symbol Device:L
- removed U3: LM2574N-5, Package_DIP:DIP-8_W7.62mm, symbol Regulator_Switching:LM2574N-5
- added BT1: Battery_Cell, symbol Device:Battery_Cell
- added C1, C2: C_Small, symbol Device:C_Small
- added PS1: TPS61023, CONV_PDQ2-D5-S3-S:CONV_PDQ2-D5-S3-S, symbol PDQ2-D5-S3-S:PDQ2-D5-S3-S
- added R10, R6, R7, R8, R9: R_Small, symbol Device:R_Small
- added SW3: SW_Nidec_CAS-120A1, Button_Switch_SMD:Nidec_Copal_CAS-120A, symbol Switch:SW_Nidec_CAS-120A1
- added U4: TP4056-42-ESOP8, Package_SO:SOIC-8-1EP_3.9x4.9mm_P1.27mm_EP2.41x3.3mm_ThermalVias, symbol Battery_Management:TP4056-42-ESOP8
Connections:
- net +5V: now also C1.1, R6.1, U4.4 (V_{CC}), U4.8 (CE)
- net GND: now also BT1.2 (-), C1.2, C2.1, R7.2, R8.1, R8.2, U4.1 (TEMP), U4.3 (GND)
- new net: R7.1, U4.2 (PROG)
- new net: BT1.1 (+), C2.2, U4.5 (BAT)
- new net: R9.2, U4.6 (~{STDBY})
- new net: R6.2, U4.7 (~{CHRG})
- new net: PS1.3 (ON/OFF), SW3.2 (B)
- new net: PS1.5 (NC), PS1.8 (NC)

Commit message: Mucenje
Parts:
- removed PS1: TPS61023, CONV_PDQ2-D5-S3-S:CONV_PDQ2-D5-S3-S, symbol PDQ2-D5-S3-S:PDQ2-D5-S3-S
- removed R8: R_Small, symbol Device:R_Small
- added C3: 10u, Capacitor_SMD:C_1206_3216Metric_Pad1.33x1.80mm_HandSolder, symbol Device:C_Small
- added C4: 2 x 22u, Capacitor_THT:CP_Radial_D5.0mm_P2.00mm, symbol Device:C_Small
- added D3, D4: LED, LED_THT:LED_D5.0mm, symbol Device:LED
- added L1: 1u, Inductor_THT:L_Radial_D7.2mm_P3.00mm_Murata_1700, symbol Device:L_Small
- added R9: 100k, Resistor_SMD:R_1206_3216Metric_Pad1.30x1.75mm_HandSolder, symbol Device:R_Small
- added U3: TPS61023DRLR, footprints:DRL0006A, symbol 2025-12-11_16-22-03:TPS61023DRLR
- BT1: value Battery_Cell -> 3.7 V; footprint (none) -> Battery:BatteryHolder_Keystone_1042_1x18650; Manufacturer (none) -> EEMB; Manufacturer part number (none) -> LIR18650
- C1: value C_Small -> 10u; footprint (none) -> Capacitor_SMD:C_1206_3216Metric_Pad1.33x1.80mm_HandSolder; Manufacturer (none) -> SAMSUNG; Manufacturer part number (none) -> CL31A106KBHNNNE
- C5: renamed from C2; value C_Small -> 10u; footprint (none) -> Capacitor_SMD:C_1206_3216Metric_Pad1.33x1.80mm_HandSolder; Manufacturer (none) -> SAMSUNG; Manufacturer part number (none) -> CL31A106KBHNNNE
- R10: value R_Small -> 732k; footprint (none) -> Resistor_SMD:R_1206_3216Metric_Pad1.30x1.75mm_HandSolder; Manufacturer (none) -> ROYALOHM; Manufacturer part number (none) -> 1206S4J0473T5E
- R6: renamed from R7; value R_Small -> 1.2k; footprint (none) -> Resistor_SMD:R_1206_3216Metric_Pad1.30x1.75mm_HandSolder; Manufacturer (none) -> ROYALOHM; Manufacturer part number (none) -> 1206S4F2001T5E
- R7: renamed from R6; value R_Small -> 1k; footprint (none) -> Resistor_SMD:R_1206_3216Metric_Pad1.30x1.75mm_HandSolder; Manufacturer (none) -> ROYALOHM; Manufacturer part number (none) -> 1206S4F2001T5E
- R8: renamed from R9; value R_Small -> 1k; footprint (none) -> Resistor_SMD:R_1206_3216Metric_Pad1.30x1.75mm_HandSolder; Manufacturer (none) -> ROYALOHM; Manufacturer part number (none) -> 1206S4F2001T5E
- SW3: value SW_Nidec_CAS-120A1 -> ~
- U4: value TP4056-42-ESOP8 -> TP4056
Connections:
- net +5V: now also D3.2 (A), D4.2 (A); no longer DS1.2 (VDD), R1.1, R7.1, RV1.1, U1.18 (+5V), U2.16 (VDD)
- net BLUE: now also U1.50 (PA12); no longer U1.42 (PC6)
- net GND: now also SW3.3 (A), C3.2, C4.2, R9.2, U3.4 (GND)
- net RED: now also U1.69 (STLINK_SWO/PB3); no longer U1.40 (PC8)
- net START: now also U1.44 (PC5); no longer U1.63 (PB10)
- net +Vin: now reaches BT1.1 (+), C5.2, U4.5 (BAT)
- net +Vin: now also SW3.1 (C), C3.1, L1.1, U3.3 (VIN)
- net 5V: now reaches R10.1
- net 5V: now also DS1.2 (VDD), R1.1, RV1.1, U1.18 (+5V), U2.16 (VDD), C4.1, U3.6 (VOUT)
- net at R10.2: now also R9.1, U3.1 (FB)
- net at SW3.2 (B): now also U3.2 (EN)
- net at R8.1: now also D3.1 (K)
- new net: L1.2, U3.5 (SW)
- new net: D4.1 (K), R7.1
- no-connect marks 60 -> 61
Other:
- moved on the sheet: BT1, C1, C5, D1, D2, DS1, H1, H2, H3, H4, R1, R2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

Commit message: uprdejt
Parts:
- added J1: USB_B_Mini, Connector_USB:USB_Mini-B_Lumberg_2486_01_Horizontal, symbol Connector:USB_B_Mini
Connections:
- net 5V: now also R4.1, R5.1
- net GND: now also J1.5 (GND), J1.6 (Shield)
- net +5V renamed USB 5V
- net USB 5V: now also J1.1 (VBUS); no longer R4.1, R5.1
- no-connect marks 61 -> 64
Other:
- moved on the sheet: BT1, C1, C3, C4, C5, D3, D4, L1, R10, R5, R6, R7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

Commit message: Word
Parts:
- removed U4: TP4056, Package_SO:SOIC-8-1EP_3.9x4.9mm_P1.27mm_EP2.41x3.3mm_ThermalVias, symbol Battery_Management:TP4056-42-ESOP8
- added U4: TP4056, SOP127P600X175-9N:SOP127P600X175-9N, symbol TP4056:TP4056
- BT1: Manufacturer EEMB -> VELOG; Manufacturer part number LIR18650 -> 18650-2200mAh-3.7V
Connections:
- net +Vin: now also U4.5 (BAT)
- net GND: now also U4.1 (TEMP), U4.3 (GND), U4.9 (EP)
- net SDA: now also U1.21 (PB7); no longer U1.43 (PB9)
- net STOP: now also U1.39 (PC9); no longer U1.61 (PA8)
- net USB 5V: now also U4.4 (VCC), U4.8 (CE)
- net at R6.1: now also U4.2 (PROG)
- net CHRG: now reaches R8.2
- net CHRG: now also U4.7 (~{CHRG})
- net STDBY: now reaches R7.2
- net STDBY: now also U4.6 (~{STDBY})
- no-connect marks 64 -> 63
Other:
- moved on the sheet: BT1, C1, C5, D1, D2, D3, D4, R2, R3, R6, R7, R8
