File: Seminar.kicad_pcb (KiCad board)
At the start: 2 copper layers, 17 parts, among them SW1 SW_Push, SW2 SW_Push, U1 NUCLEO64-F446RE, U2 PCF8574AP

Commit message: Update Seminar 7.12.
Parts:
- added C1: 22u, Capacitor_THT:CP_Radial_D5.0mm_P2.00mm, F.Cu at (51.0, -19.0)
- added C2: 220u, Capacitor_THT:CP_Radial_D5.0mm_P2.00mm, F.Cu at (38.6, -19.0)
- added D3: 11DQ06TA, Diode_THT:D_DO-41_SOD81_P12.70mm_Horizontal, F.Cu at (39.2, -10.0)
- added J1: Screw_Terminal_01x02, TerminalBlock_MetzConnect:TerminalBlock_MetzConnect_Type011_RT05502HBLC_1x02_P5.00mm_Horizontal, F.Cu at (43.5, -35.9)
- added L1: 330u, Inductor_THT:L_Radial_D7.2mm_P3.00mm_Murata_1700, F.Cu at (61.5, -0.50)
- added U3: LM2574N-5, Package_DIP:DIP-8_W7.62mm, F.Cu at (34.7, 9.30)
- moved RV1 39.8 mm to (12.7, 5.30)
- moved U2 39.8 mm to (-6.92, 1.50)
- moved R5 36.9 mm to (-36.9, -1.50), turned to 180 degrees
- moved R4 33.0 mm to (-36.9, 1.80), turned to 180 degrees
- moved R3 29.4 mm to (-36.9, 5.12), turned to 180 degrees
- moved R2 26.1 mm to (-36.9, 8.43), turned to 180 degrees
- moved SW1 24.4 mm to (-79.0, -36.5)
- moved SW2 24.4 mm to (-79.2, -19.8)
- moved R1 23.3 mm to (-36.9, 11.7), turned to 180 degrees
- moved D1 22.0 mm to (-70.0, 3.50)
- moved D2 19.4 mm to (-52.0, 4.00)
- moved DS1 12.0 mm to (12.5, -12.1)

Commit message: Update Seminar 7.12. dva
Parts:
- RV1: footprint Potentiometer_SMD:Potentiometer_ACP_CA6-VSMD_Vertical -> Potentiometer_THT:Potentiometer_Bourns_3299Y_Vertical
- moved RV1 3.34 mm to (15.5, 3.50)
Changed lines of the file:
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@@
 		)
 	)
-	(footprint "Potentiometer_SMD:Potentiometer_ACP_CA6-VSMD_Vertical"
+	(footprint "Potentiometer_THT:Potentiometer_Bourns_3299Y_Vertical"
 		(layer "F.Cu")
-		(at 12.69 5.305)
-		(descr "Potentiometer, vertical, ACP CA6-VSMD, http://www.acptechnologies.com/wp-content/uploads/2017/06/01-ACP-CA6.pdf")
-		(tags "Potentiometer vertical ACP CA6-VSMD")
+		(at 15.5 3.5)
+		(descr "Potentiometer, vertical, Bourns 3299Y, https://www.bourns.com/pdfs/3299.pdf")
+		(tags "Potentiometer vertical Bourns 3299Y")
 		(property "Reference" "RV1"
-			(at 0 -4.5 0)
+			(at -2.54 -3.16 0)
 			(layer "F.SilkS")
 			(effects
@@
 		)
 		(property "Value" "R_Potentiometer_Small"
-			(at 0 4.5 0)
+			(at -2.54 5.44 0)
 			(layer "F.Fab")
 			(effects
@@
 		(sheetname "/")
 		(sheetfile "Seminar.kicad_sch")
-		(attr smd)
-		(fp_line
-			(start -3.36 0.92)
-			(end -3.36 -0.92)
-			(stroke
-				(width 0.12)
-				(type solid)
-			)
-			(layer "F.SilkS")
-		)
-		(fp_line
-			(start -2.845 -3.36)
-			(end 3.36 -3.36)
-			(stroke
-				(width 0.12)
-				(type solid)
-			)
-			(layer "F.SilkS")
-		)
-		(fp_line
-			(start 3.36 -3.36)
-			(end 3.36 -1.23)
-			(stroke
-				(width 0.12)
-				(type solid)
-			)
-			(layer "F.SilkS")
-		)
-		(fp_line
-			(start 3.36 1.23)
-			(end 3.36 3.36)
-			(stroke
-				(width 0.12)
-				(type solid)
-			)
-			(layer "F.SilkS")
-		)
-		(fp_line
-			(start 3.36 3.36)
-			(end -2.845 3.36)
+		(attr through_hole)
+		(fp_line
+			(start -7.415 -2.02)
+			(end 2.335 -2.02)
+			(stroke
+				(width 0.12)
+				(type solid)
+			)
+			(layer "F.SilkS")
+		)
+		(fp_line
+			(start -7.415 4.3)
+			(end -7.415 -2.02)
+			(stroke
+				(width 0.12)
+				(type solid)
+			)
+			(layer "F.SilkS")
+		)
+		(fp_line
+			(start 2.335 -2.02)
+			(end 2.335 4.3)
+			(stroke
+				(width 0.12)
+				(type solid)
+			)
+			(layer "F.SilkS")
+		)
+		(fp_line
+			(start 2.335 4.3)
+			(end -7.415 4.3)
 			(stroke
 				(width 0.12)
@@
 		)
 		(fp_rect
-			(start -5.83 -3.5)
-			(end 5.83 3.51)
+			(start -7.56 -2.16)
+			(end 2.48 4.44)
 			(stroke
 				(width 0.05)
@@
 			(layer "F.CrtYd")
 		)
+		(fp_line
+			(start 1.652 2.09)
+			(end 0.125 3.617)
+			(stroke
+				(width 0.1)
+				(type solid)
+			)
+			(layer "F.Fab")
+		)
+		(fp_line
+			(start 1.785 2.223)
+			(end 0.258 3.75)
+			(stroke
+				(width 0.1)
+				(type solid)
+			)
+			(layer "F.Fab")
+		)
 		(fp_rect
-			(start -3.25 -3.25)
-			(end 3.25 3.25)
+			(start -7.305 -1.91)
+			(end 2.225 4.19)
 			(stroke
 				(width 0.1)
@@
 		)
 		(fp_circle
-			(center 0.275 0)
-			(end 1.175 0)
+			(center 0.955 2.92)
+			(end 2.05 2.92)
 			(stroke
 				(width 0.1)
@@
 		)
 		(fp_text user "${REFERENCE}"
-			(at -2.25 0 90)
-			(layer "F.Fab")
-			(effects
-				(font
-					(size 1 1)
-					(thickness 0.15)
-				)
-			)
-		)
-		(pad "1" smd roundrect
-			(at -4.325 2.15)
-			(size 2.5 2)
-			(layers "F.Cu" "F.Mask" "F.Paste")
-			(roundrect_rratio 0.125)
+			(at -3.175 1.14 0)
+			(layer "F.Fab")
+			(effects
+				(font
+					(size 1 1)
+					(thickness 0.15)
+				)
+			)
+		)
+		(pad "1" thru_hole circle
+			(at 0 0)
+			(size 1.44 1.44)
+			(drill 0.8)
+			(layers "*.Cu" "*.Mask")
+			(remove_unused_layers no)
 			(net 17 "+5V")
 			(pinfunction "1")
 			(pintype "passive")
 		)
-		(pad "2" smd roundrect
-			(at 4.325 0)
-			(size 2.5 2)
-			(layers "F.Cu" "F.Mask" "F.Paste")
-			(roundrect_rratio 0.125)
+		(pad "2" thru_hole circle
+			(at -2.54 2.54)
+			(size 1.44 1.44)
+			(drill 0.8)
+			(layers "*.Cu" "*.Mask")
+			(remove_unused_layers no)
 			(net 6 "Net-(DS1-VO)")
 			(pinfunction "2")
 			(pintype "passive")
 		)
-		(pad "3" smd roundrect
-			(at -4.325 -2.15)
-			(size 2.5 2)
-			(layers "F.Cu" "F.Mask" "F.Paste")
-			(roundrect_rratio 0.125)
+		(pad "3" thru_hole circle
+			(at -5.08 0)
+			(size 1.44 1.44)
+			(drill 0.8)
+			(layers "*.Cu" "*.Mask")
+			(remove_unused_layers no)
 			(net 1 "GND")
 			(pinfunction "3")
@@
 		)
 		(embedded_fonts no)
-		(model "${KICAD9_3DMODEL_DIR}/Potentiometer_SMD.3dshapes/Potentiometer_ACP_CA6-VSMD_Vertical.step"
+		(model "${KICAD9_3DMODEL_DIR}/Potentiometer_THT.3dshapes/Potentiometer_Bourns_3299Y_Vertical.step"
 			(offset
 				(xyz 0 0 0)

Commit message: Mucenje
Parts:
- added BT1: 3.7 V, Battery:BatteryHolder_Keystone_1042_1x18650, F.Cu at (-168.6, -17.8)
- added C1: 10u, Capacitor_SMD:C_1206_3216Metric_Pad1.33x1.80mm_HandSolder, F.Cu at (-157.8, 25.3)
- added C3: 10u, Capacitor_SMD:C_1206_3216Metric_Pad1.33x1.80mm_HandSolder, F.Cu at (-169.5, 16.4)
- added C4: 2 x 22u, Capacitor_THT:CP_Radial_D5.0mm_P2.00mm, F.Cu at (-140.8, 27.1)
- added C5: 10u, Capacitor_SMD:C_1206_3216Metric_Pad1.33x1.80mm_HandSolder, F.Cu at (-148.3, 17.7)
- added D3: LED, LED_THT:LED_D5.0mm, F.Cu at (-167.8, 24.1)
- added D4: LED, LED_THT:LED_D5.0mm, F.Cu at (-169.2, 1.33)
- added L1: 1u, Inductor_THT:L_Radial_D7.2mm_P3.00mm_Murata_1700, F.Cu at (-138.8, 14.2)
- added R10: 732k, Resistor_SMD:R_1206_3216Metric_Pad1.30x1.75mm_HandSolder, F.Cu at (-125.2, -1.00)
- added R6: 1.2k, Resistor_SMD:R_1206_3216Metric_Pad1.30x1.75mm_HandSolder, F.Cu at (-180.5, 6.69)
- added R7: 1k, Resistor_SMD:R_1206_3216Metric_Pad1.30x1.75mm_HandSolder, F.Cu at (-156.2, 6.81)
- added R8: 1k, Resistor_SMD:R_1206_3216Metric_Pad1.30x1.75mm_HandSolder, F.Cu at (-163.4, 20.8)
- added R9: 100k, Resistor_SMD:R_1206_3216Metric_Pad1.30x1.75mm_HandSolder, F.Cu at (-132.2, 6.00)
- added SW3: ~, Button_Switch_SMD:Nidec_Copal_CAS-120A, F.Cu at (-145.6, 7.00)
- added U3: TPS61023, footprints:DRL0006A, F.Cu at (-125.1, 5.77)
- added U4: TP4056, Package_SO:SOIC-8-1EP_3.9x4.9mm_P1.27mm_EP2.41x3.3mm_ThermalVias, F.Cu at (-169.4, 9.02)
- moved J1 257.9 mm to (-205.0, 33.3)
- moved C1 250.8 mm to (-196.8, 19.6)
- moved L1 235.8 mm to (-171.5, 35.8)
- moved D3 233.4 mm to (-191.5, 25.4), turned to -90 degrees
- moved C2 219.8 mm to (-171.3, 46.3)
- moved U3 212.7 mm to (-176.9, 30.6), turned to 180 degrees
- moved RV1 170.3 mm to (-151.2, 38.3)
- moved R2 167.9 mm to (-198.2, 55.1), turned to 90 degrees
- moved R5 153.9 mm to (-179.8, 55.6)
- moved R3 153.9 mm to (-179.8, 62.1), turned to 90 degrees
- moved H3 148.2 mm to (-222.0, 168.2)
- moved DS1 145.7 mm to (-116.1, 56.3), turned to 90 degrees
- moved R4 142.6 mm to (-168.3, 57.1), turned to -90 degrees
- moved D2 140.0 mm to (-185.3, 46.9)
- moved U2 139.5 mm to (-133.8, 59.7), turned to 180 degrees
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Connections:
- DS1 pad 2: +5V -> 5V
- R1 pad 1: +5V -> 5V
- RV1 pad 1: +5V -> 5V
- U1 pad 18: +5V -> 5V
- U1 pad 40: RED -> unconnected-(U1-PC8-Pad40)
- U1 pad 42: BLUE -> unconnected-(U1-PC6-Pad42)
- U1 pad 44: unconnected-(U1-PC5-Pad44) -> START
- U1 pad 50: unconnected-(U1-PA12-Pad50) -> BLUE
- U1 pad 63: START -> unconnected-(U1-PB10-Pad63)
- U1 pad 69: unconnected-(U1-STLINK_SWO/PB3-Pad69) -> RED
- U2 pad 16: +5V -> 5V
Routing:
- net GND: track 0.00 -> 174.8 mm, vias 0 -> 4
- net 5V: track 0.00 -> 131.0 mm
- net +Vin: track 0.00 -> 99.4 mm
- net +5V: track 0.00 -> 98.2 mm
- net Net-(D3-K): track 0.00 -> 46.5 mm, vias 0 -> 2
- net Net-(DS1-D7): track 0.00 -> 44.3 mm
- net Net-(DS1-VO): track 0.00 -> 43.9 mm
- net Net-(DS1-D4): track 0.00 -> 41.6 mm
- net Net-(DS1-D6): track 0.00 -> 37.9 mm
- net Net-(DS1-D5): track 0.00 -> 31.9 mm
- net START: track 0.00 -> 30.0 mm
- net VD: track 0.00 -> 29.0 mm
- net STOP: track 0.00 -> 26.0 mm
- net SDA: track 0.00 -> 25.2 mm
- net SCL: track 0.00 -> 23.1 mm
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- added copper zone on B.Cu, net GND

Commit message: update 3d model
Parts:
- moved H3 420.5 mm to (198.5, 168.8), turned to 90 degrees
- moved R2 325.8 mm to (112.5, 153.2), turned to 180 degrees
- moved H1 322.1 mm to (24.8, 168.8), turned to 90 degrees
- moved D1 317.2 mm to (104.3, 150.6), turned to -90 degrees
- moved SW2 314.6 mm to (113.0, 144.0), turned to 0 degrees
- moved R3 308.0 mm to (119.5, 134.8), turned to 180 degrees
- moved C1 304.0 mm to (77.0, 151.8), turned to 90 degrees
- moved D2 303.5 mm to (104.4, 137.3), turned to 90 degrees
- moved R5 303.4 mm to (113.0, 134.9), turned to -90 degrees
- moved D3 299.9 mm to (82.8, 146.6), turned to 0 degrees
- moved J1 293.1 mm to (63.2, 151.7)
- moved R4 290.4 mm to (114.5, 123.3), turned to 0 degrees
- moved H4 288.1 mm to (198.5, 23.5), turned to 90 degrees
- moved C2 286.4 mm to (103.7, 126.3), turned to 90 degrees
- moved SW1 284.7 mm to (116.0, 117.6), turned to 180 degrees
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Routing:
- net VD: track 29.0 -> 23.4 mm
- net Net-(U3-FB): track 10.4 -> 12.1 mm
- net START: track 30.0 -> 28.5 mm
- net Net-(D2-A): track 14.9 -> 13.6 mm
- net Net-(D4-K): track 14.6 -> 13.4 mm
- net GND: track 174.8 -> 175.7 mm
Other:
- board outline added: 185.7 x 157.2 mm

Commit message: uprdejt
Parts:
- added J1: USB_B_Mini, Connector_USB:USB_Mini-B_Lumberg_2486_01_Horizontal, F.Cu at (63.2, 146.1)
- U3: value TPS61023 -> TPS61023DRLR
- moved C1 21.9 mm to (74.5, 130.0), turned to -90 degrees
- moved J1 21.7 mm to (60.5, 130.1)
- moved BT1 17.2 mm to (38.8, 106.5)
- moved R6 17.0 mm to (63.9, 118.2)
- moved R3 14.0 mm to (117.3, 121.0)
- moved C3 14.0 mm to (71.6, 110.7)
- moved C4 14.0 mm to (82.3, 82.0)
- moved C5 14.0 mm to (72.9, 89.5)
- moved D1 14.0 mm to (102.1, 136.8)
- moved D3 14.0 mm to (80.6, 132.8)
- moved D4 14.0 mm to (56.4, 109.2)
- moved R10 14.0 mm to (54.2, 66.5)
- moved R4 14.0 mm to (112.3, 109.5)
- moved R8 14.0 mm to (76.0, 104.6)
- moved R9 14.0 mm to (61.2, 73.5)
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Connections:
- C1 pad 1: +5V -> USB 5V
- D3 pad 2: +5V -> USB 5V
- D4 pad 2: +5V -> USB 5V
- R4 pad 1: +5V -> 5V
- R5 pad 1: +5V -> 5V
- U4 pad 4: +5V -> USB 5V
- U4 pad 8: +5V -> USB 5V
Routing:
- net USB 5V: track 0.00 -> 38.4 mm, vias 0 -> 2
- net +Vin: track 99.4 -> 70.9 mm
- net SDA: track 25.2 -> 0.00 mm
- net SCL: track 23.1 -> 0.00 mm
- net +5V: track 97.8 -> 77.1 mm
- net GND: track 175.7 -> 156.6 mm
- net BLUE: track 17.9 -> 0.00 mm
- net RED: track 17.0 -> 0.00 mm
- net START: track 28.5 -> 12.0 mm
- net STOP: track 26.0 -> 14.1 mm
- net VD: track 23.4 -> 14.8 mm
- net 5V: track 131.0 -> 139.6 mm
- net Net-(U4-PROG): track 8.56 -> 5.56 mm

Commit message: Word
Parts:
- U4: footprint Package_SO:SOIC-8-1EP_3.9x4.9mm_P1.27mm_EP2.41x3.3mm_ThermalVias -> SOP127P600X175-9N:SOP127P600X175-9N
- moved J1 37.0 mm to (97.2, 126.2), turned to 180 degrees
- moved C3 34.9 mm to (53.0, 81.2), turned to 90 degrees
- moved SW2 27.7 mm to (110.8, 102.5), turned to 90 degrees
- moved SW1 23.8 mm to (115.2, 80.0), turned to -90 degrees
- moved D1 21.1 mm to (118.2, 123.2), turned to 180 degrees
- moved J1 21.0 mm to (62.8, 125.1)
- moved R5 19.3 mm to (105.7, 102.5), turned to 0 degrees
- moved R4 18.8 mm to (104.2, 92.5)
- moved C2 17.3 mm to (91.1, 98.7)
- moved H1 13.6 mm to (24.8, 155.2), turned to 180 degrees
- moved H3 13.6 mm to (198.5, 155.2), turned to 180 degrees
- moved R2 11.5 mm to (117.2, 130.2)
- moved R3 10.3 mm to (108.0, 116.8)
- moved U2 9.13 mm to (115.3, 65.9)
- moved RV1 7.97 mm to (96.9, 85.3), turned to -90 degrees
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Connections:
- R7 pad 2: Net-(U4-~{CHRG}) -> STDBY
- R8 pad 2: Net-(U4-~{STDBY}) -> CHRG
- U1 pad 21: unconnected-(U1-PB7-Pad21) -> SDA
- U1 pad 39: unconnected-(U1-PC9-Pad39) -> STOP
- U1 pad 43: SDA -> unconnected-(U1-PB9-Pad43)
- U1 pad 61: STOP -> unconnected-(U1-PA8-Pad61)
- U4 pad 6: Net-(U4-~{STDBY}) -> STDBY
- U4 pad 7: Net-(U4-~{CHRG}) -> CHRG
Routing:
- net +5V: track 77.1 -> 16.5 mm, vias 0 -> 2
- net SCL: track 0.00 -> 39.7 mm, vias 0 -> 2
- net START: track 12.0 -> 46.5 mm
- net USB 5V: track 38.4 -> 65.7 mm
- net Net-(DS1-D4): track 41.6 -> 21.4 mm
- net BLUE: track 0.00 -> 19.3 mm
- net +Vin: track 70.9 -> 88.2 mm
- net SDA: track 0.00 -> 15.8 mm
- net RED: track 0.00 -> 14.8 mm
- net 5V: track 139.6 -> 126.7 mm
- net Net-(DS1-VO): track 43.9 -> 32.7 mm, vias 0 -> 2
- net STOP: track 14.1 -> 25.2 mm
- net Net-(U4-~{STDBY}): track 11.1 -> 0.00 mm
- net Net-(U4-~{CHRG}): track 10.8 -> 0.00 mm
- net CHRG: track 0.00 -> 10.4 mm, vias 0 -> 2
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Other:
- board size 185.7 x 157.2 mm -> 185.8 x 143.8 mm

Commit message: Finito
Parts:
- removed the D3 at (83.1, 126.3)
- removed the J1 at (97.2, 126.2)
- SW3: value ~ -> SPDT; footprint Button_Switch_SMD:Nidec_Copal_CAS-120A -> Button_Switch_THT:SW_Slide_SPDT_Straight_CK_OS102011MS2Q
- moved J1 28.8 mm to (63.0, 153.8)
- moved SW3 3.92 mm to (60.2, 90.2)
- moved C1 3.49 mm to (84.3, 96.9)
- moved C2 3.49 mm to (93.8, 101.0)
- moved C5 3.49 mm to (73.4, 94.6)
- moved D3 3.49 mm to (82.0, 106.1)
- moved L1 3.49 mm to (93.7, 109.8)
- moved R7 3.49 mm to (65.4, 101.0)
- moved D4 3.49 mm to (59.6, 107.7)
- moved R8 3.49 mm to (78.8, 101.7)
- moved U4 3.49 mm to (70.8, 108.5)
- moved R6 3.49 mm to (71.6, 115.5)
- moved U3 3.49 mm to (88.5, 115.3)
- moved C1 3.15 mm to (72.2, 127.8)
- moved R3 3.07 mm to (105.0, 116.0)
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Routing:
- net USB 5V: track 65.7 -> 91.4 mm
- net VD: track 23.9 -> 12.8 mm
- net GND: track 147.6 -> 137.6 mm, vias 2 -> 0
- net Net-(D3-K): track 40.4 -> 34.6 mm
- net Net-(SW3-B): track 15.8 -> 19.4 mm, vias 0 -> 2
- net +Vin: track 88.2 -> 90.5 mm
- net BLUE: track 19.3 -> 21.6 mm
- net RED: track 14.8 -> 12.9 mm
- net unconnected-(U1-PA11-Pad52): track 0.00 -> 1.63 mm
- net Net-(D2-A): track 6.51 -> 7.35 mm
Other:
- board size 185.8 x 143.8 mm -> 185.8 x 142 mm

Commit message: PCB Update
Parts:
- U1: footprint Module:ST_Morpho_Connector_144_STLink -> STM32F446RET6:QFP50P1200X1200X160-64N
- moved H4 63.4 mm to (135.1, 23.4)
- moved H3 63.4 mm to (135.2, 153.6)
- moved U1 49.4 mm to (118.8, 103.2), turned to 180 degrees
- moved SW1 41.6 mm to (108.0, 121.0), turned to 90 degrees
- moved R2 41.0 mm to (116.8, 89.2), turned to 90 degrees
- moved D2 39.2 mm to (127.8, 90.5), turned to 90 degrees
- moved D1 33.7 mm to (110.3, 90.5), turned to 90 degrees
- moved R3 31.3 mm to (121.3, 89.2), turned to 90 degrees
- moved R5 25.1 mm to (130.8, 104.3), turned to -90 degrees
- moved SW2 21.8 mm to (129.0, 114.5), turned to -90 degrees
- moved R4 12.0 mm to (106.8, 104.2), turned to -90 degrees
- moved H2 9.93 mm to (34.7, 23.4)
- moved H1 9.93 mm to (34.7, 153.6)
- moved C1 6.48 mm to (89.6, 93.1)
- moved R6 6.48 mm to (76.8, 111.7)
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Connections:
- U1 pad 17: unconnected-(U1-PA15-Pad17) -> BLUE
- U1 pad 23: unconnected-(U1-PC13-Pad23) -> RED
- U1 pad 39: STOP -> unconnected-(U1-PC9-Pad39)
- U1 pad 4: unconnected-(U1-PD2-Pad4) -> STOP
- U1 pad 50: BLUE -> unconnected-(U1-PA12-Pad50)
Routing:
- net GND: track 137.6 -> 170.5 mm
- net START: track 46.5 -> 22.4 mm
- net BLUE: track 21.6 -> 7.29 mm
- net 5V: track 126.7 -> 140.1 mm, vias 0 -> 2
- net SDA: track 15.8 -> 28.9 mm
- net RED: track 12.9 -> 7.91 mm
- net STOP: track 25.2 -> 22.3 mm
- net SCL: track 39.7 -> 37.9 mm
- net unconnected-(U1-PA11-Pad52): track 1.63 -> 0.00 mm
- net Net-(D2-A): track 7.35 -> 6.62 mm
Other:
- board size 185.8 x 142 mm -> 112.1 x 141.8 mm
- board text added: "CHRG"
- board text added: "Ivan Hodak"
- board text added: "MIN"
- board text added: "SEK"
- board text added: "START"
- board text added: "STDBY"
- board text added: "STOP"
- board text added: "Štoperica v1.0"
