File: Seminar.kicad_pcb (KiCad board)
At the start: 2 copper layers, 112.1 x 141.8 mm, 38 parts, among them J1 USB_B_Mini, SW1 SW_Push, SW2 SW_Push, SW3 SPDT, U1 NUCLEO64-F446RE, U2 PCF8574AP, U3 LM2574N-5, U3 TPS61023DRLR, U4 TP4056

Commit message: a
Connections:
- U1 pad 18: 5V -> GND
- U1 pad 19: GND -> 5V
- U1 pad 20: GND -> unconnected-(U1-PA4-Pad20)
- U1 pad 22: GND -> unconnected-(U1-PA6-Pad22)
- U1 pad 31: unconnected-(U1-PH1-Pad31) -> GND
- U1 pad 32: unconnected-(U1-PA4-Pad32) -> 5V
- U1 pad 48: unconnected-(U1-NC-Pad48) -> 5V
- U1 pad 58: GND -> unconnected-(U1-PB6-Pad58)
- U1 pad 63: unconnected-(U1-PB10-Pad63) -> GND
- U1 pad 64: unconnected-(U1-PB15-Pad64) -> 5V
- U1 pad 8: GND -> unconnected-(U1-PC0-Pad8)
Routing:
- net GND: track 170.5 -> 157.8 mm
- net 5V: track 140.1 -> 149.0 mm, vias 2 -> 0
- net unconnected-(U1-PB6-Pad58): track 0.00 -> 0.81 mm

Commit message: dorada
Parts:
- moved J1 0.30 mm to (68.2, 149.8), turned to 0 degrees
Routing:
- net GND: track 157.8 -> 185.1 mm, vias 0 -> 2
- net 5V: track 149.0 -> 167.3 mm, vias 0 -> 4
- net USB 5V: track 91.4 -> 86.8 mm

Commit message: Dorada
Parts:
- removed the C1 at (77.5, 124.0)
- removed the C1 at (89.6, 93.1)
- removed C2: 220u, Capacitor_THT:CP_Radial_D5.0mm_P2.00mm
- removed the L1 at (99.0, 106.0)
- removed the L1 at (76.5, 79.2)
- removed the U3 at (93.8, 111.5)
- removed the U3 at (68.0, 65.6)
- added C1: 10u, Capacitor_SMD:C_1206_3216Metric_Pad1.33x1.80mm_HandSolder, F.Cu at (103.2, 84.3)
- added L1: 1u, Inductor_THT:L_Radial_D7.2mm_P3.00mm_Murata_1700, F.Cu at (105.2, 95.5)
- added U3: TPS61023DRLR, footprints:SOT563-ORI, F.Cu at (114.8, 93.5)
- moved H2 158.3 mm to (190.9, 49.2)
- moved R10 131.5 mm to (192.6, 73.2), turned to 180 degrees
- moved H4 130.9 mm to (190.6, 142.0)
- moved R9 124.4 mm to (192.6, 76.5), turned to 180 degrees
- moved R7 122.7 mm to (192.6, 83.1), turned to 180 degrees
- moved H1 119.0 mm to (91.9, 49.2), turned to 0 degrees
- moved R6 118.5 mm to (192.6, 86.4), turned to 180 degrees
- moved R8 110.1 mm to (192.6, 79.8)
- moved BT1 108.2 mm to (141.4, 55.5), turned to 0 degrees
- moved R1 86.6 mm to (158.5, 107.0), turned to 0 degrees
- moved R4 86.5 mm to (192.6, 93.0), turned to 180 degrees
- moved R2 76.5 mm to (192.6, 99.7), turned to 180 degrees
- moved D4 72.5 mm to (131.8, 75.8), turned to 180 degrees
- moved R3 71.7 mm to (192.6, 96.4), turned to 180 degrees
- moved J1 69.9 mm to (92.7, 84.2), turned to -90 degrees
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Routing:
- net GND: track 185.1 -> 0.00 mm, vias 2 -> 0
- net 5V: track 167.3 -> 0.00 mm, vias 4 -> 0
- net +Vin: track 90.5 -> 0.00 mm
- net USB 5V: track 86.8 -> 0.00 mm, vias 2 -> 0
- net SCL: track 38.0 -> 0.00 mm, vias 2 -> 0
- net Net-(DS1-D7): track 34.9 -> 0.00 mm
- net Net-(D3-K): track 34.6 -> 0.00 mm
- net Net-(DS1-VO): track 32.7 -> 0.00 mm, vias 2 -> 0
- net Net-(DS1-D6): track 30.5 -> 0.00 mm
- net SDA: track 28.9 -> 0.00 mm
- net Net-(DS1-D5): track 26.3 -> 0.00 mm
- net START: track 22.4 -> 0.00 mm
- net STOP: track 22.3 -> 0.00 mm
- net Net-(DS1-D4): track 21.4 -> 0.00 mm
- net Net-(SW3-B): track 19.8 -> 0.00 mm, vias 2 -> 0
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Other:
- board size 112.1 x 141.8 mm -> 111.2 x 105 mm
- board text removed: "Ivan Hodak"
- board text removed: "Štoperica v1.0"

Commit message: dorada
Parts:
- moved R9 84.2 mm to (109.2, 88.8)
- moved R10 82.0 mm to (113.5, 94.8), turned to 90 degrees
- moved R7 77.1 mm to (117.0, 68.0)
- moved R6 61.7 mm to (131.2, 79.5), turned to 0 degrees
- moved R8 61.5 mm to (131.2, 84.5)
- moved R2 40.1 mm to (156.3, 82.8), turned to 90 degrees
- moved R3 37.0 mm to (156.3, 89.2), turned to 90 degrees
- moved R5 18.3 mm to (176.0, 97.5), turned to 90 degrees
- moved R4 18.2 mm to (176.0, 85.5), turned to 90 degrees
- moved C5 14.2 mm to (107.3, 73.0), turned to 0 degrees
- moved D3 12.6 mm to (136.3, 73.0)
- moved R1 9.36 mm to (167.8, 105.8), turned to -90 degrees
- moved U4 7.68 mm to (116.8, 75.7)
- moved U3 5.08 mm to (119.8, 92.8)
- moved C1 4.59 mm to (107.8, 83.5)
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Routing:
- net GND: track 0.00 -> 158.9 mm, vias 0 -> 6
- net 5V: track 0.00 -> 148.1 mm, vias 0 -> 2
- net USB 5V: track 0.00 -> 46.7 mm
- net +Vin: track 0.00 -> 42.5 mm
- net STOP: track 0.00 -> 41.6 mm, vias 0 -> 2
- net Net-(DS1-RS): track 0.00 -> 40.2 mm
- net START: track 0.00 -> 35.7 mm
- net Net-(DS1-R/W): track 0.00 -> 34.0 mm
- net SCL: track 0.00 -> 28.3 mm, vias 0 -> 6
- net Net-(DS1-E): track 0.00 -> 27.4 mm
- net SDA: track 0.00 -> 26.9 mm, vias 0 -> 2
- net Net-(DS1-LED(+)): track 0.00 -> 26.1 mm
- net CHRG: track 0.00 -> 23.9 mm
- net Net-(U3-SW): track 0.00 -> 16.9 mm, vias 0 -> 2
- net Net-(D2-A): track 0.00 -> 15.3 mm, vias 0 -> 2
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Other:
- board size 111.2 x 105 mm -> 104.5 x 105 mm
- board text added: "Ivan Hodak"
- board text added: "Štoperica v2"

Commit message: Final
Parts:
- moved U1 3.57 mm to (141.0, 87.8)
- moved R2 2.49 mm to (154.0, 83.8)
- moved R3 2.47 mm to (154.0, 90.2)
Routing:
- net +Vin: track 42.5 -> 72.7 mm, vias 0 -> 2
- net GND: track 158.9 -> 155.0 mm, vias 6 -> 8
- net START: track 35.7 -> 39.3 mm
- net SDA: track 26.9 -> 29.2 mm
- net 5V: track 148.1 -> 146.0 mm
- net Net-(D2-A): track 15.3 -> 17.0 mm
- net RED: track 7.81 -> 8.90 mm
- net STOP: track 41.6 -> 40.6 mm
- net BLUE: track 7.10 -> 8.05 mm
- net SCL: track 28.3 -> 29.0 mm
