File: Seminar.kicad_pcb (KiCad board)
At the start: 2 copper layers, 104.5 x 105 mm, 34 parts, among them J1 USB_B_Mini, SW1 SW_Push, SW2 SW_Push, SW3 SPDT, U1 NUCLEO64-F446RE, U2 PCF8574AP, U3 TPS61023DRLR, U4 TP4056

Commit message: FINAL
Parts:
- moved BT1 4.14 mm to (145.8, 55.5)
Routing:
- net +Vin: track 72.7 -> 73.3 mm
Changed lines of the file:
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@@
 	(footprint "Battery:BatteryHolder_Keystone_1042_1x18650"
 		(layer "F.Cu")
-		(at 141.610106 55.5)
+		(at 145.75 55.5)
 		(descr "Battery holder, Keystone 1042, battery type 1x18650, http://www.keyelco.com/product.cfm/product_id/918, generated with kicad-footprint-generator StandardBox_generator.py")
 		(tags "horizontal single")
 		(property "Reference" "BT1"
-			(at 3.56 -11.28 0)
+			(at -0.69 -11.53 0)
 			(layer "F.SilkS")
 			(effects
@@
 		)
 		(property "Value" "3.7 V"
-			(at 0.139894 11.78 0)
+			(at -4.110106 11.53 0)
 			(layer "F.Fab")
 			(effects
@@
 		(attr smd)
 		(fp_line
-			(start -35.33 -10.435)
-			(end 35.75 -10.435)
+			(start -39.58 -10.685)
+			(end 31.5 -10.685)
+			(stroke
+				(width 0.12)
+				(type solid)
+			)
+			(layer "F.SilkS")
+		)
+		(fp_line
+			(start -39.58 10.685)
+			(end -39.58 3.51)
 			(stroke
 				(width 0.12)
@@
 		)
 		(fp_line
-			(start -35.33 10.935)
-			(end -35.33 3.76)
+			(start 31.5 -10.685)
+			(end 31.5 -3.325)
 			(stroke
 				(width 0.12)
@@
 		)
 		(fp_line
-			(start 35.75 -10.435)
-			(end 35.75 -3.075)
+			(start 31.5 3.51)
+			(end 31.5 10.685)
 			(stroke
 				(width 0.12)
@@
 		)
 		(fp_line
-			(start 35.75 3.76)
-			(end 35.75 10.935)
+			(start 31.5 10.685)
+			(end -39.58 10.685)
 			(stroke
 				(width 0.12)
@@
 		)
 		(fp_line
-			(start 35.75 10.935)
-			(end -35.33 10.935)
-			(stroke
-				(width 0.12)
-				(type solid)
-			)
-			(layer "F.SilkS")
-		)
-		(fp_line
-			(start -40.38 -3.5)
-			(end -35.47 -3.5)
+			(start -44.63 -3.75)
+			(end -39.72 -3.75)
 			(stroke
 				(width 0.05)
@@
 		)
 		(fp_line
-			(start -40.38 4)
-			(end -40.38 -3.5)
+			(start -44.63 3.75)
+			(end -44.63 -3.75)
 			(stroke
 				(width 0.05)
@@
 		)
 		(fp_line
-			(start -35.47 -10.58)
-			(end 36 -10.58)
+			(start -39.72 -10.83)
+			(end 31.75 -10.83)
 			(stroke
 				(width 0.05)
@@
 		)
 		(fp_line
-			(start -35.47 -3.5)
-			(end -35.47 -10.58)
+			(start -39.72 -3.75)
+			(end -39.72 -10.83)
 			(stroke
 				(width 0.05)
@@
 		)
 		(fp_line
-			(start -35.47 4)
-			(end -40.38 4)
+			(start -39.72 3.75)
+			(end -44.63 3.75)
 			(stroke
 				(width 0.05)
@@
 		)
 		(fp_line
-			(start -35.47 11.08)
-			(end -35.47 4)
+			(start -39.72 10.83)
+			(end -39.72 3.75)
 			(stroke
 				(width 0.05)
@@
 		)
 		(fp_line
-			(start 36 -10.58)
-			(end 36 -3.53)
+			(start 31.75 -10.83)
+			(end 31.75 -3.78)
 			(stroke
 				(width 0.05)
@@
 		)
 		(fp_line
-			(start 36 -3.53)
-			(end 40.75 -3.53)
+			(start 31.75 -3.78)
+			(end 36.5 -3.78)
 			(stroke
 				(width 0.05)
@@
 		)
 		(fp_line
-			(start 36 3.97)
-			(end 36 11.08)
+			(start 31.75 3.72)
+			(end 31.75 10.83)
 			(stroke
 				(width 0.05)
@@
 		)
 		(fp_line
-			(start 36 11.08)
-			(end -35.47 11.08)
+			(start 31.75 10.83)
+			(end -39.72 10.83)
 			(stroke
 				(width 0.05)
@@
 		)
 		(fp_line
-			(start 40.75 -3.53)
-			(end 40.75 3.97)
+			(start 36.5 -3.78)
+			(end 36.5 3.72)
 			(stroke
 				(width 0.05)
@@
 		)
 		(fp_line
-			(start 40.75 3.97)
-			(end 36 3.97)
+			(start 36.5 3.72)
+			(end 31.75 3.72)
 			(stroke
 				(width 0.05)
@@
 		)
 		(fp_rect
-			(start -35.25 -10.075)
-			(end 35.56 10.575)
+			(start -39.5 -10.325)
+			(end 31.31 10.325)
 			(stroke
 				(width 0.1)
@@
 		)
 		(fp_text user "+"
-			(at -36.44 -4.75 0)
+			(at -40.69 -5 0)
 			(layer "F.SilkS")
 			(effects
@@
 		)
 		(fp_text user "+"
-			(at -31.44 0.1 0)
+			(at -35.69 -0.15 0)
 			(layer "F.Fab")
 			(effects
@@
 		)
 		(fp_text user "${REFERENCE}"
-			(at 3.56 0.25 0)
+			(at -0.69 0 0)
 			(layer "F.Fab")
 			(effects
@@
 		)
 		(pad "" np_thru_hole circle
-			(at -32.57 -7.75)
+			(at -35.75 -8)
 			(size 2.39 2.39)
 			(drill 2.39)
@@
 		)
 		(pad "" np_thru_hole circle
-			(at -24.06 8.25)
+			(at -27.75 7.5)
 			(size 3.45 3.45)
 			(drill 3.45)
@@
 		)
 		(pad "" np_thru_hole circle
-			(at 31.18 -7.75)
-			(size 3.45 3.45)
+			(at 27.5 -7.5)
+			(size 3.29539 3.29539)
 			(drill 3.45)
 			(layers "*.Cu" "*.Mask")
 		)
 		(pad "1" smd roundrect
-			(at -36.13 0.25)
+			(at -40.38 0)
 			(size 7.5 6.5)
 			(layers "F.Cu" "F.Mask" "F.Paste")
@@
 		)
 		(pad "2" smd roundrect
-			(at 36.5 0.25)
+			(at 32.25 0)
 			(size 7.5 6.5)
 			(layers "F.Cu" "F.Mask" "F.Paste")
@@
 			)
 			(scale
-				(xyz 0.9 0.9 1)
+				(xyz 1 1 1)
 			)
 			(rotate
@@
 	)
 	(segment
+		(start 155.225 73.25)
+		(end 172.975 55.5)
+		(width 1)
+		(layer "F.Cu")
+		(net 1)
+	)
+	(segment
 		(start 99.475 85.15)
 		(end 107.7375 85.15)
@@
 	)
 	(segment
-		(start 172.725 55.75)
-		(end 178.110106 55.75)
-		(width 1)
-		(layer "F.Cu")
-		(net 1)
-	)
-	(segment
 		(start 116.5 83.225)
 		(end 116.574 83.299)
@@
 	)
 	(segment
-		(start 155.225 73.25)
-		(end 172.725 55.75)
-		(width 1)
-		(layer "F.Cu")
-		(net 1)
-	)
-	(segment
 		(start 137.701 82.947324)
 		(end 137.701 82.07)
@@
 	)
 	(segment
+		(start 172.975 55.5)
+		(end 178 55.5)
+		(width 1)
+		(layer "F.Cu")
+		(net 1)
+	)
+	(segment
 		(start 121.5 94.5)
 		(end 121.95 94.5)
@@
 	)
 	(segment
-		(start 108.8375 72.6625)
-		(end 105.480106 69.305106)
-		(width 1)
-		(layer "F.Cu")
-		(net 75)
-	)
-	(segment
 		(start 111.33397 79.677)
 		(end 117.913339 79.677)
@@
 	)
 	(segment
+		(start 105.37 55.5)
+		(end 105.37 69.5325)
+		(width 1)
+		(layer "F.Cu")
+		(net 75)
+	)
+	(segment
 		(start 127.525 88.6875)
 		(end 122.9625 88.6875)
@@
 	)
 	(segment
-		(start 105.480106 69.305106)
-		(end 105.480106 55.75)
+		(start 105.37 69.5325)
+		(end 108.8375 73)
 		(width 1)
 		(layer "F.Cu")
@@
 	(segment
 		(start 114.241364 88.75)
+		(end 116.991364 91.5)
+		(width 0.3)
+		(layer "F.Cu")
+		(net 80)
+	)
+	(segment
+		(start 114.241364 88.75)
 		(end 110.8 88.75)
 		(width 0.3)
@@
 	)
 	(segment
-		(start 117.275 92.275)
-		(end 117.275 91.783636)
+		(start 116.991364 91.5)
+		(end 118.05 91.5)
 		(width 0.3)
 		(layer "F.Cu")
@@
 		(width 0.3)
 		(layer "F.Cu")
-		(net 80)
-	)
-	(segment
-		(start 117.275 91.783636)
-		(end 114.241364 88.75)
-		(width 0.3)
-		(layer "F.Cu")
